Commit message: updated grasping and gripper packages

File: apc_gripper_position/urdf/gripper.xacro (robot description, xacro)
@@ -52,9 +52,9 @@
       <inertial>
         <mass value="0.1" />
-        <origin rpy="0 0 ${pi}" xyz="-0.0622 0 0" />
+        <origin rpy="0 0 ${pi}" xyz="0 0 0" />
         <inertia ixx="0.0000847702" ixy="0" ixz="0" iyy="0.0000955040" iyz="0" izz="0.0000331406" />
       </inertial>
       <collision>
-        <origin rpy="0 0 ${pi}" xyz="-0.0622 0 0" />
+        <origin rpy="0 0 ${pi}" xyz="0 0 0" />
         <geometry>
           <mesh filename="package://apc_gripper_position/meshes/mesh_dedo_eslabon.stl" scale="0.001 0.001 0.001"/>
@@ -62,5 +62,5 @@
       </collision>
       <visual>
-        <origin rpy="0 0 ${pi}" xyz="-0.0622 0 0" />
+        <origin rpy="0 0 ${pi}" xyz="0 0 0" />
         <geometry>
           <mesh filename="package://apc_gripper_position/meshes/mesh_dedo_eslabon.stl" scale="0.001 0.001 0.001"/>

File: apc_gripper_position/urdf/joints.xacro (robot description, xacro)
@@ -5,5 +5,5 @@
       <axis xyz="0 1 0" />
       <limit effort="1000" lower="-0.1" upper="0.1" velocity="0.5" />
-      <origin rpy="0 0 0" xyz="0.0311 -0.046785 0.093" />
+      <origin rpy="0 0 0" xyz="0.0 -0.046785 0.101" />
       <parent link="gripper_body" />
       <child link="left_ext" />
@@ -22,5 +22,5 @@
       <axis xyz="0 1 0" />
       <limit effort="1000" lower="-0.1" upper="0.1" velocity="0.5" />
-      <origin rpy="0 0 0" xyz="0.0311 0.046785 0.093" />
+      <origin rpy="0 0 0" xyz="0.0 0.046785 0.101" />
       <parent link="gripper_body" />
       <child link="right_ext" />
