Commit message: fixed gripper simulation

File: apc_gripper/urdf/gripper_old.xacro (robot description, xacro)
@@ -7,5 +7,5 @@
       <inertial>
         <mass value="0.1" />
-        <origin rpy="0 0 0" xyz="0 0 0" />
+        <origin rpy="0 0 0" xyz="0 0 0.063" />
         <inertia ixx="0.13292157" ixy="0.0" ixz="0" iyy="0.8980362" iyz="0" izz="0.6991288" />
       </inertial>
@@ -21,6 +21,6 @@
           <mesh filename="package://apc_gripper/meshes/mesh_soporte.stl" scale="0.001 0.001 0.001"/>
         </geometry>
-        <material name="gris">
-         <color rgba="0.5 0.5 0.5 1"/>
+        <material name="blug">
+         <color rgba="0 1 1 1"/>
         </material>
       </visual>
@@ -30,6 +30,6 @@
     <inertial>
       <mass value="0.1" />
-      <origin rpy="0 0 0" xyz="0 0 0" />
-      <inertia ixx="0.0000847702" ixy="0" ixz="0" iyy="0.0000955040" iyz="0" izz="0.0000331406" />
+      <origin rpy="0 0 0" xyz="-0.031 0 0.04" />
+      <inertia ixx="0.0000213613" ixy="0" ixz="0" iyy="0.0000595838" iyz="0" izz="0.0000394382" />
     </inertial>
       <collision>
@@ -44,6 +44,6 @@
           <mesh filename="package://apc_gripper/meshes/mesh_eslabon.stl" scale="0.001 0.001 0.001"/>
         </geometry>
-        <material name="blu">
-         <color rgba="0 0 1 1"/>
+        <material name="blug">
+         <color rgba="0 1 1 1"/>
         </material>
       </visual>
@@ -74,10 +74,10 @@
     <inertial>
       <mass value="0.1" />
-      <origin rpy="0 0 0" xyz="0 0 0" />
-      <inertia ixx="0.0000847702" ixy="0" ixz="0" iyy="0.0000955040" iyz="0" izz="0.0000331406" />
+      <origin rpy="0 0 0" xyz="-0.031 0 0.04" />
+      <inertia ixx="0.0000213613" ixy="0" ixz="0" iyy="0.0000595838" iyz="0" izz="0.0000394382" />
     </inertial>
-    <collision>
-      <origin rpy="0 0 0" xyz="0 0 0" />
-      <geometry>
+      <collision>
+        <origin rpy="0 0 0" xyz="0 0 0" />
+        <geometry>
           <mesh filename="package://apc_gripper/meshes/mesh_eslabon.stl" scale="0.001 0.001 0.001"/>
         </geometry>
@@ -88,6 +88,6 @@
           <mesh filename="package://apc_gripper/meshes/mesh_eslabon.stl" scale="0.001 0.001 0.001"/>
         </geometry>
-        <material name="blu">
-         <color rgba="0 0 1 1"/>
+        <material name="blug">
+         <color rgba="0 1 1 1"/>
         </material>
       </visual>
@@ -164,8 +164,8 @@
   <!-- END - Robot description -->
   <!-- Used for fixing robot to Gazebo 'base_link' -->
-  <!-- <link name="world"/>
+  <link name="world"/>
   <joint name="fixed" type="fixed">
     <parent link="world"/>
     <child link="gripper_body"/>
-  </joint> -->
+  </joint>
 </robot>

File: apc_gripper/urdf/joints.xacro (robot description, xacro)
@@ -4,5 +4,5 @@
     <joint name="gripper_body__left_ext" type="revolute">
       <axis xyz="1 0 0" />
-      <limit effort="1000" lower="-3.14" upper="3.14" velocity="0.5" />
+      <limit effort="1000" lower="-0.15" upper="0.8" velocity="0.5" />
       <origin rpy="0 0 0" xyz="0.0311 -0.046785 0.093" />
       <parent link="gripper_body" />
@@ -10,12 +10,12 @@
     </joint>
     <transmission name="trans_gripper_body__left_ext">
-      <type>transmission_interface/SimpleTransmission</type>
-      <joint name="gripper_body__left_ext">
-        <hardwareInterface>hardware_interface/EffortJointInterface</hardwareInterface>
-      </joint>
-      <actuator name="motor_gripper_body__left_ext">
-        <hardwareInterface>hardware_interface/EffortJointInterface</hardwareInterface>
-        <mechanicalReduction>1</mechanicalReduction>
-      </actuator>
+  		<type>transmission_interface/SimpleTransmission</type>
+  		<joint name="gripper_body__left_ext">
+  			<hardwareInterface>hardware_interface/PositionJointInterface</hardwareInterface>
+  		</joint>
+  		<actuator name="motor_gripper_body__left_ext">
+  			<hardwareInterface>hardware_interface/PositionJointInterface</hardwareInterface>
+  			<mechanicalReduction>1</mechanicalReduction>
+  		</actuator>
     </transmission>
     <joint name="gripper_body__left_int" type="revolute">
@@ -25,15 +25,6 @@
       <parent link="gripper_body" />
       <child link="left_int" />
+      <mimic joint="gripper_body__left_ext" multiplier="1" offset="0" />
     </joint>
-    <transmission name="trans_gripper_body__left_int">
-      <type>transmission_interface/SimpleTransmission</type>
-      <joint name="gripper_body__left_int">
-        <hardwareInterface>hardware_interface/EffortJointInterface</hardwareInterface>
-      </joint>
-      <actuator name="motor_gripper_body__left_int">
-        <hardwareInterface>hardware_interface/EffortJointInterface</hardwareInterface>
-        <mechanicalReduction>1</mechanicalReduction>
-      </actuator>
-    </transmission>
     <joint name="gripper_body__right_ext" type="revolute">
       <axis xyz="1 0 0" />
@@ -42,15 +33,6 @@
       <parent link="gripper_body" />
       <child link="right_ext" />
+      <mimic joint="gripper_body__left_ext" multiplier="-1" offset="0" />
     </joint>
-    <transmission name="trans_gripper_body__right_ext">
-      <type>transmission_interface/SimpleTransmission</type>
-      <joint name="gripper_body__right_ext">
-        <hardwareInterface>hardware_interface/EffortJointInterface</hardwareInterface>
-      </joint>
-      <actuator name="motor_gripper_body__right_ext">
-        <hardwareInterface>hardware_interface/EffortJointInterface</hardwareInterface>
-        <mechanicalReduction>1</mechanicalReduction>
-      </actuator>
-    </transmission>
     <joint name="gripper_body__right_int" type="revolute">
       <axis xyz="1 0 0" />
@@ -59,4 +41,5 @@
       <parent link="gripper_body" />
       <child link="right_int" />
+      <mimic joint="gripper_body__right_ext" multiplier="1" offset="0" />
     </joint>
   <!-- FINGERS -->
@@ -68,15 +51,6 @@
       <parent link="left_ext" />
       <child link="left_finger" />
+      <mimic joint="gripper_body__left_ext" multiplier="-1" offset="0" />
     </joint>
-    <transmission name="trans_left_ext__left_finger">
-      <type>transmission_interface/SimpleTransmission</type>
-      <joint name="left_ext__left_finger">
-        <hardwareInterface>hardware_interface/EffortJointInterface</hardwareInterface>
-      </joint>
-      <actuator name="motor_left_ext__left_finger">
-        <hardwareInterface>hardware_interface/EffortJointInterface</hardwareInterface>
-        <mechanicalReduction>1</mechanicalReduction>
-      </actuator>
-    </transmission>
   <!-- RIGHT FINGER -->
       <joint name="right_ext__right_finger" type="revolute">
@@ -86,4 +60,5 @@
       <parent link="right_ext" />
       <child link="right_finger" />
+      <mimic joint="gripper_body__right_ext" multiplier="-1" offset="0" />
     </joint>
   <!-- END - Robot description -->

File: irb140_sim/urdf/irb140.xacro (robot description, xacro)
@@ -8,5 +8,6 @@
   <xacro:include filename="$(find irb140_sim)/urdf/irb140.gazebo"/>
 	<!-- gripper files -->
-	<xacro:include filename="$(find apc_gripper_position)/urdf/gripper.xacro"/>
+	<!-- <xacro:include filename="$(find apc_gripper_position)/urdf/gripper.xacro"/> -->
+	<xacro:include filename="$(find apc_gripper)/urdf/gripper.xacro"/>
  	<!--LINKS-->
 	<!--base_link-->

File: irb140_sim/urdf/irb140_joints.xacro (robot description, xacro)
@@ -136,5 +136,5 @@
 		<parent link="link_6"/>
 		<child link="tcp_link"/>
-		<origin rpy="0 0 0" xyz="0.20 0 0"/>
+		<origin rpy="0 0 0" xyz="0.21 0 0"/>
 	</joint>
 </robot>
