Commit message: changed to latest gripper model

File: apc_gripper/urdf/gripper.xacro (robot description, xacro)
@@ -13,5 +13,5 @@
         <origin rpy="0 0 0" xyz="0 0 0" />
         <geometry>
-          <mesh filename="package://apc_gripper/meshes/mesh_soporte.stl" scale="0.001 0.001 0.001"/>
+          <mesh filename="package://apc_gripper/meshes/mesh_cuerpo.stl" scale="0.001 0.001 0.001"/>
         </geometry>
       </collision>
@@ -19,5 +19,5 @@
         <origin rpy="0 0 0" xyz="0 0 0" />
         <geometry>
-          <mesh filename="package://apc_gripper/meshes/mesh_soporte.stl" scale="0.001 0.001 0.001"/>
+          <mesh filename="package://apc_gripper/meshes/mesh_cuerpo.stl" scale="0.001 0.001 0.001"/>
         </geometry>
         <material name="gris">
@@ -36,5 +36,5 @@
         <origin rpy="0 0 0" xyz="0 0 0" />
         <geometry>
-          <mesh filename="package://apc_gripper/meshes/mesh_eslabon.stl" scale="0.001 0.001 0.001"/>
+          <mesh filename="package://apc_gripper/meshes/mesh_eslabon_externo.stl" scale="0.001 0.001 0.001"/>
         </geometry>
       </collision>
@@ -42,5 +42,5 @@
         <origin rpy="0 0 0" xyz="0 0 0" />
         <geometry>
-          <mesh filename="package://apc_gripper/meshes/mesh_eslabon.stl" scale="0.001 0.001 0.001"/>
+          <mesh filename="package://apc_gripper/meshes/mesh_eslabon_externo.stl" scale="0.001 0.001 0.001"/>
         </geometry>
         <material name="blu">
@@ -58,5 +58,5 @@
         <origin rpy="0 0 0" xyz="0 0 0" />
         <geometry>
-          <mesh filename="package://apc_gripper/meshes/mesh_eslabon.stl" scale="0.001 0.001 0.001"/>
+          <mesh filename="package://apc_gripper/meshes/mesh_eslabon_interno.stl" scale="0.001 0.001 0.001"/>
         </geometry>
       </collision>
@@ -64,5 +64,5 @@
         <origin rpy="0 0 0" xyz="0 0 0" />
         <geometry>
-          <mesh filename="package://apc_gripper/meshes/mesh_eslabon.stl" scale="0.001 0.001 0.001"/>
+          <mesh filename="package://apc_gripper/meshes/mesh_eslabon_interno.stl" scale="0.001 0.001 0.001"/>
         </geometry>
         <material name="blug">
@@ -80,5 +80,5 @@
       <origin rpy="0 0 0" xyz="0 0 0" />
       <geometry>
-          <mesh filename="package://apc_gripper/meshes/mesh_eslabon.stl" scale="0.001 0.001 0.001"/>
+          <mesh filename="package://apc_gripper/meshes/mesh_eslabon_externo.stl" scale="0.001 0.001 0.001"/>
         </geometry>
       </collision>
@@ -86,5 +86,5 @@
         <origin rpy="0 0 0" xyz="0 0 0" />
         <geometry>
-          <mesh filename="package://apc_gripper/meshes/mesh_eslabon.stl" scale="0.001 0.001 0.001"/>
+          <mesh filename="package://apc_gripper/meshes/mesh_eslabon_externo.stl" scale="0.001 0.001 0.001"/>
         </geometry>
         <material name="blu">
@@ -102,5 +102,5 @@
         <origin rpy="0 0 0" xyz="0 0 0" />
         <geometry>
-          <mesh filename="package://apc_gripper/meshes/mesh_eslabon.stl" scale="0.001 0.001 0.001"/>
+          <mesh filename="package://apc_gripper/meshes/mesh_eslabon_interno.stl" scale="0.001 0.001 0.001"/>
         </geometry>
       </collision>
@@ -108,5 +108,5 @@
         <origin rpy="0 0 0" xyz="0 0 0" />
         <geometry>
-          <mesh filename="package://apc_gripper/meshes/mesh_eslabon.stl" scale="0.001 0.001 0.001"/>
+          <mesh filename="package://apc_gripper/meshes/mesh_eslabon_interno.stl" scale="0.001 0.001 0.001"/>
         </geometry>
         <material name="blug">
@@ -120,9 +120,9 @@
     <inertial>
       <mass value="0.1" />
-      <origin rpy="0 0 0" xyz="-0.031 0.018 0.032" />
+      <origin rpy="0 0 0" xyz="0 0.018 0.032" />
       <inertia ixx="0.0000847702" ixy="0" ixz="0" iyy="0.0000955040" iyz="0" izz="0.0000331406" />
     </inertial>
       <collision>
-        <origin rpy="0 0 0" xyz="0 0 0" />
+        <origin rpy="0 0 0" xyz="0 -0.002 0" />
         <geometry>
           <mesh filename="package://apc_gripper/meshes/mesh_dedo.stl" scale="0.001 0.001 0.001"/>
@@ -143,9 +143,9 @@
   <inertial>
     <mass value="0.1" />
-    <origin rpy="0 0 ${pi}" xyz="-0.031 -0.018 0.032" />
+    <origin rpy="0 0 ${pi}" xyz="0 -0.018 0.032" />
     <inertia ixx="0.0000847702" ixy="0" ixz="0" iyy="0.0000955040" iyz="0" izz="0.0000331406" />
   </inertial>
       <collision>
-        <origin rpy="0 0 ${pi}" xyz="-0.0620 0 0" />
+        <origin rpy="0 0 0" xyz="0 -0.002 0.0" />
         <geometry>
           <mesh filename="package://apc_gripper/meshes/mesh_dedo.stl" scale="0.001 0.001 0.001"/>
@@ -153,5 +153,5 @@
       </collision>
       <visual>
-        <origin rpy="0 0 ${pi}" xyz="-0.0620 0 0" />
+        <origin rpy="0 0 0" xyz="0 0 0" />
         <geometry>
           <mesh filename="package://apc_gripper/meshes/mesh_dedo.stl" scale="0.001 0.001 0.001"/>

File: apc_gripper/urdf/joints.xacro (robot description, xacro)
@@ -5,5 +5,5 @@
       <axis xyz="1 0 0" />
       <limit effort="1000" lower="-0.15" upper="0.8" velocity="0.5" />
-      <origin rpy="0 0 0" xyz="0.0311 -0.046785 0.093" />
+      <origin rpy="0 0 0" xyz="0.0 -0.046785 0.103" />
       <parent link="gripper_body" />
       <child link="left_ext" />
@@ -22,5 +22,5 @@
       <axis xyz="1 0 0" />
       <limit effort="1000" lower="-3.14" upper="3.14" velocity="0.5" />
-      <origin rpy="0 0 0" xyz="0.0311 -0.026 0.105" />
+      <origin rpy="0 0 0" xyz="0.0 -0.026 0.115" />
       <parent link="gripper_body" />
       <child link="left_int" />
@@ -30,16 +30,16 @@
       <axis xyz="1 0 0" />
       <limit effort="1000" lower="-3.14" upper="3.14" velocity="0.5" />
-      <origin rpy="0 0 0" xyz="0.0311 0.046785 0.093" />
+      <origin rpy="0 0 3.14" xyz="0 0.046785 0.103" />
       <parent link="gripper_body" />
       <child link="right_ext" />
-      <mimic joint="gripper_body__left_ext" multiplier="-1" offset="0" />
+      <mimic joint="gripper_body__left_ext" multiplier="1" offset="0" />
     </joint>
     <joint name="gripper_body__right_int" type="revolute">
       <axis xyz="1 0 0" />
       <limit effort="1000" lower="-3.14" upper="3.14" velocity="0.5" />
-      <origin rpy="0 0 0" xyz="0.0311 0.026 0.105" />
+      <origin rpy="0 0 0" xyz="0.0 0.026 0.115" />
       <parent link="gripper_body" />
       <child link="right_int" />
-      <mimic joint="gripper_body__right_ext" multiplier="1" offset="0" />
+      <mimic joint="gripper_body__right_ext" multiplier="-1" offset="0" />
     </joint>
   <!-- FINGERS -->

Commit message: formatting

File: apc_gripper/urdf/gripper.xacro (robot description, xacro)
@@ -1,29 +1,29 @@
-<?xml version="1.0" ?>
+<?xml version="1.0"?>
 <robot name="gripper" xmlns:xacro="http://ros.org/wiki/xacro">
-<xacro:include filename="$(find apc_gripper)/urdf/joints.xacro"/>
-<xacro:include filename="$(find apc_gripper)/urdf/gripper.gazebo"/>
+  <xacro:include filename="$(find apc_gripper)/urdf/joints.xacro" />
+  <xacro:include filename="$(find apc_gripper)/urdf/gripper.gazebo" />
   <!-- BASE LINK -->
-    <link name="gripper_body">
-      <inertial>
-        <mass value="0.1" />
-        <origin rpy="0 0 0" xyz="0 0 0" />
-        <inertia ixx="0.13292157" ixy="0.0" ixz="0" iyy="0.8980362" iyz="0" izz="0.6991288" />
-      </inertial>
-      <collision>
-        <origin rpy="0 0 0" xyz="0 0 0" />
-        <geometry>
-          <mesh filename="package://apc_gripper/meshes/mesh_cuerpo.stl" scale="0.001 0.001 0.001"/>
-        </geometry>
-      </collision>
-      <visual>
-        <origin rpy="0 0 0" xyz="0 0 0" />
-        <geometry>
-          <mesh filename="package://apc_gripper/meshes/mesh_cuerpo.stl" scale="0.001 0.001 0.001"/>
-        </geometry>
-        <material name="gris">
-         <color rgba="0.5 0.5 0.5 1"/>
-        </material>
-      </visual>
-    </link>
+  <link name="gripper_body">
+    <inertial>
+      <mass value="0.1" />
+      <origin rpy="0 0 0" xyz="0 0 0" />
+      <inertia ixx="0.13292157" ixy="0.0" ixz="0" iyy="0.8980362" iyz="0" izz="0.6991288" />
+    </inertial>
+    <collision>
+      <origin rpy="0 0 0" xyz="0 0 0" />
+      <geometry>
+        <mesh filename="package://apc_gripper/meshes/mesh_cuerpo.stl" scale="0.001 0.001 0.001" />
+      </geometry>
+    </collision>
+    <visual>
+      <origin rpy="0 0 0" xyz="0 0 0" />
+      <geometry>
+        <mesh filename="package://apc_gripper/meshes/mesh_cuerpo.stl" scale="0.001 0.001 0.001" />
+      </geometry>
+      <material name="gris">
+        <color rgba="0.5 0.5 0.5 1" />
+      </material>
+    </visual>
+  </link>
   <!-- LINKS -->
   <link name="left_ext">
@@ -33,20 +33,20 @@
       <inertia ixx="0.0000847702" ixy="0" ixz="0" iyy="0.0000955040" iyz="0" izz="0.0000331406" />
     </inertial>
-      <collision>
-        <origin rpy="0 0 0" xyz="0 0 0" />
-        <geometry>
-          <mesh filename="package://apc_gripper/meshes/mesh_eslabon_externo.stl" scale="0.001 0.001 0.001"/>
-        </geometry>
-      </collision>
-      <visual>
-        <origin rpy="0 0 0" xyz="0 0 0" />
-        <geometry>
-          <mesh filename="package://apc_gripper/meshes/mesh_eslabon_externo.stl" scale="0.001 0.001 0.001"/>
-        </geometry>
-        <material name="blu">
-         <color rgba="0 0 1 1"/>
-        </material>
-      </visual>
-    </link>
+    <collision>
+      <origin rpy="0 0 0" xyz="0 0 0" />
+      <geometry>
+        <mesh filename="package://apc_gripper/meshes/mesh_eslabon_externo.stl" scale="0.001 0.001 0.001" />
+      </geometry>
+    </collision>
+    <visual>
+      <origin rpy="0 0 0" xyz="0 0 0" />
+      <geometry>
+        <mesh filename="package://apc_gripper/meshes/mesh_eslabon_externo.stl" scale="0.001 0.001 0.001" />
+      </geometry>
+      <material name="blu">
+        <color rgba="0 0 1 1" />
+      </material>
+    </visual>
+  </link>
   <link name="left_int">
     <inertial>
@@ -55,20 +55,20 @@
       <inertia ixx="0.0000213613" ixy="0" ixz="0" iyy="0.0000595838" iyz="0" izz="0.0000394382" />
     </inertial>
-      <collision>
-        <origin rpy="0 0 0" xyz="0 0 0" />
-        <geometry>
-          <mesh filename="package://apc_gripper/meshes/mesh_eslabon_interno.stl" scale="0.001 0.001 0.001"/>
-        </geometry>
-      </collision>
-      <visual>
-        <origin rpy="0 0 0" xyz="0 0 0" />
-        <geometry>
-          <mesh filename="package://apc_gripper/meshes/mesh_eslabon_interno.stl" scale="0.001 0.001 0.001"/>
-        </geometry>
-        <material name="blug">
-         <color rgba="0 1 1 1"/>
-        </material>
-      </visual>
-    </link>
+    <collision>
+      <origin rpy="0 0 0" xyz="0 0 0" />
+      <geometry>
+        <mesh filename="package://apc_gripper/meshes/mesh_eslabon_interno.stl" scale="0.001 0.001 0.001" />
+      </geometry>
+    </collision>
+    <visual>
+      <origin rpy="0 0 0" xyz="0 0 0" />
+      <geometry>
+        <mesh filename="package://apc_gripper/meshes/mesh_eslabon_interno.stl" scale="0.001 0.001 0.001" />
+      </geometry>
+      <material name="blug">
+        <color rgba="0 1 1 1" />
+      </material>
+    </visual>
+  </link>
   <link name="right_ext">
     <inertial>
@@ -80,17 +80,17 @@
       <origin rpy="0 0 0" xyz="0 0 0" />
       <geometry>
-          <mesh filename="package://apc_gripper/meshes/mesh_eslabon_externo.stl" scale="0.001 0.001 0.001"/>
-        </geometry>
-      </collision>
-      <visual>
-        <origin rpy="0 0 0" xyz="0 0 0" />
-        <geometry>
-          <mesh filename="package://apc_gripper/meshes/mesh_eslabon_externo.stl" scale="0.001 0.001 0.001"/>
-        </geometry>
-        <material name="blu">
-         <color rgba="0 0 1 1"/>
-        </material>
-      </visual>
-    </link>
+        <mesh filename="package://apc_gripper/meshes/mesh_eslabon_externo.stl" scale="0.001 0.001 0.001" />
+      </geometry>
+    </collision>
+    <visual>
+      <origin rpy="0 0 0" xyz="0 0 0" />
+      <geometry>
+        <mesh filename="package://apc_gripper/meshes/mesh_eslabon_externo.stl" scale="0.001 0.001 0.001" />
+      </geometry>
+      <material name="blu">
+        <color rgba="0 0 1 1" />
+      </material>
+    </visual>
+  </link>
   <link name="right_int">
     <inertial>
@@ -99,20 +99,20 @@
       <inertia ixx="0.0000213613" ixy="0" ixz="0" iyy="0.0000595838" iyz="0" izz="0.0000394382" />
     </inertial>
-      <collision>
-        <origin rpy="0 0 0" xyz="0 0 0" />
-        <geometry>
-          <mesh filename="package://apc_gripper/meshes/mesh_eslabon_interno.stl" scale="0.001 0.001 0.001"/>
-        </geometry>
-      </collision>
-      <visual>
-        <origin rpy="0 0 0" xyz="0 0 0" />
-        <geometry>
-          <mesh filename="package://apc_gripper/meshes/mesh_eslabon_interno.stl" scale="0.001 0.001 0.001"/>
-        </geometry>
-        <material name="blug">
-         <color rgba="0 1 1 1"/>
-        </material>
-      </visual>
-    </link>
+    <collision>
+      <origin rpy="0 0 0" xyz="0 0 0" />
+      <geometry>
+        <mesh filename="package://apc_gripper/meshes/mesh_eslabon_interno.stl" scale="0.001 0.001 0.001" />
+      </geometry>
+    </collision>
+    <visual>
+      <origin rpy="0 0 0" xyz="0 0 0" />
+      <geometry>
+        <mesh filename="package://apc_gripper/meshes/mesh_eslabon_interno.stl" scale="0.001 0.001 0.001" />
+      </geometry>
+      <material name="blug">
+        <color rgba="0 1 1 1" />
+      </material>
+    </visual>
+  </link>
   <!-- FINGERS -->
   <!-- LEFT FINGER -->
@@ -123,43 +123,45 @@
       <inertia ixx="0.0000847702" ixy="0" ixz="0" iyy="0.0000955040" iyz="0" izz="0.0000331406" />
     </inertial>
-      <collision>
-        <origin rpy="0 0 0" xyz="0 -0.002 0" />
-        <geometry>
-          <mesh filename="package://apc_gripper/meshes/mesh_dedo.stl" scale="0.001 0.001 0.001"/>
-        </geometry>
-      </collision>
-      <visual>
-        <origin rpy="0 0 0" xyz="0 0 0" />
-        <geometry>
-          <mesh filename="package://apc_gripper/meshes/mesh_dedo.stl" scale="0.001 0.001 0.001"/>
-        </geometry>
-        <material name="white">
-         <color rgba="1 1 1 1"/>
-        </material>
-      </visual>
-    </link>
+    <collision>
+      <!-- <origin rpy="0 0 0" xyz="0 -0.002 0" /> -->
+      <origin rpy="0 0 0" xyz="0 0 0" />
+      <geometry>
+        <mesh filename="package://apc_gripper/meshes/mesh_dedo.stl" scale="0.001 0.001 0.001" />
+      </geometry>
+    </collision>
+    <visual>
+      <origin rpy="0 0 0" xyz="0 0 0" />
+      <geometry>
+        <mesh filename="package://apc_gripper/meshes/mesh_dedo.stl" scale="0.001 0.001 0.001" />
+      </geometry>
+      <material name="white">
+        <color rgba="1 1 1 1" />
+      </material>
+    </visual>
+  </link>
   <!-- RIGHT FINGER -->
-<link name="right_finger">
-  <inertial>
-    <mass value="0.1" />
-    <origin rpy="0 0 ${pi}" xyz="0 -0.018 0.032" />
-    <inertia ixx="0.0000847702" ixy="0" ixz="0" iyy="0.0000955040" iyz="0" izz="0.0000331406" />
-  </inertial>
-      <collision>
-        <origin rpy="0 0 0" xyz="0 -0.002 0.0" />
-        <geometry>
-          <mesh filename="package://apc_gripper/meshes/mesh_dedo.stl" scale="0.001 0.001 0.001"/>
-        </geometry>
-      </collision>
-      <visual>
-        <origin rpy="0 0 0" xyz="0 0 0" />
-        <geometry>
-          <mesh filename="package://apc_gripper/meshes/mesh_dedo.stl" scale="0.001 0.001 0.001"/>
-        </geometry>
-        <material name="white">
-         <color rgba="1 1 1 1"/>
-        </material>
-      </visual>
-    </link>
+  <link name="right_finger">
+    <inertial>
+      <mass value="0.1" />
+      <origin rpy="0 0 ${pi}" xyz="0 0.018 0.032" />
+      <inertia ixx="0.0000847702" ixy="0" ixz="0" iyy="0.0000955040" iyz="0" izz="0.0000331406" />
+    </inertial>
+    <collision>
+      <!-- <origin rpy="0 0 0" xyz="0 -0.002 0.0" /> -->
+      <origin rpy="0 0 0" xyz="0 0 0" />
+      <geometry>
+        <mesh filename="package://apc_gripper/meshes/mesh_dedo.stl" scale="0.001 0.001 0.001" />
+      </geometry>
+    </collision>
+    <visual>
+      <origin rpy="0 0 0" xyz="0 0 0" />
+      <geometry>
+        <mesh filename="package://apc_gripper/meshes/mesh_dedo.stl" scale="0.001 0.001 0.001" />
+      </geometry>
+      <material name="white">
+        <color rgba="1 1 1 1" />
+      </material>
+    </visual>
+  </link>
   <!-- END - Robot description -->
   <!-- Used for fixing robot to Gazebo 'base_link' -->

File: irb140_sim/urdf/irb140_joints.xacro (robot description, xacro)
@@ -1,14 +1,14 @@
-<?xml version="1.0" ?>
+<?xml version="1.0"?>
 <robot xmlns:xacro="http://ros.org/wiki/xacro">
- 	<!--Joints-->
+	<!--Joints-->
 	<!--joint_1-->
 	<joint name="joint_1" type="revolute">
-    <origin rpy="0 0 0" xyz="0 0 0"/>
-    <parent link="base_link"/>
-    <child link="link_1"/>
-    <axis xyz="0 0 1"/>
-    <limit effort="1000" lower="-3.1416" upper="3.1416" velocity="2.618"/>
-  </joint>
-  <transmission name="trans_joint_1">
+		<origin rpy="0 0 0" xyz="0 0 0" />
+		<parent link="base_link" />
+		<child link="link_1" />
+		<axis xyz="0 0 1" />
+		<limit effort="1000" lower="-3.1416" upper="3.1416" velocity="2.618" />
+	</joint>
+	<transmission name="trans_joint_1">
 		<type>transmission_interface/SimpleTransmission</type>
 		<joint name="joint_1">
@@ -19,14 +19,14 @@
 			<mechanicalReduction>1</mechanicalReduction>
 		</actuator>
-  </transmission>
+	</transmission>
 	<!--joint_2-->
 	<joint name="joint_2" type="revolute">
-    <origin rpy="0 0 0" xyz="0.070 0 0.352"/>
-    <parent link="link_1"/>
-    <child link="link_2"/>
-    <axis xyz="0 1 0"/>
-    <limit effort="1000" lower="-0.7853" upper="1.5708" velocity="2.618"/>
-  </joint>
-  <transmission name="trans_joint_2">
+		<origin rpy="0 0 0" xyz="0.070 0 0.352" />
+		<parent link="link_1" />
+		<child link="link_2" />
+		<axis xyz="0 1 0" />
+		<limit effort="1000" lower="-0.7853" upper="1.5708" velocity="2.618" />
+	</joint>
+	<transmission name="trans_joint_2">
 		<type>transmission_interface/SimpleTransmission</type>
 		<joint name="joint_2">
@@ -37,14 +37,14 @@
 			<mechanicalReduction>1</mechanicalReduction>
 		</actuator>
-  </transmission>
+	</transmission>
 	<!--joint_3-->
 	<joint name="joint_3" type="revolute">
-    <origin rpy="0 0 0" xyz="0 -0.065 0.360"/>
-    <parent link="link_2"/>
-    <child link="link_3"/>
-    <axis xyz="0 1 0"/>
-    <limit effort="1000" lower="-2.4434" upper="0.8726" velocity="2.618"/>
-  </joint>
-  <transmission name="trans_joint_3">
+		<origin rpy="0 0 0" xyz="0 -0.065 0.360" />
+		<parent link="link_2" />
+		<child link="link_3" />
+		<axis xyz="0 1 0" />
+		<limit effort="1000" lower="-2.4434" upper="0.8726" velocity="2.618" />
+	</joint>
+	<transmission name="trans_joint_3">
 		<type>transmission_interface/SimpleTransmission</type>
 		<joint name="joint_3">
@@ -55,14 +55,14 @@
 			<mechanicalReduction>1</mechanicalReduction>
 		</actuator>
-  </transmission>
+	</transmission>
 	<!--joint_4-->
 	<joint name="joint_4" type="revolute">
-    <origin rpy="0 0 0" xyz="0.239 0.065 0"/>
-    <parent link="link_3"/>
-    <child link="link_4"/>
-    <axis xyz="1 0 0"/>
-    <limit effort="1000" lower="-3.49" upper="3.49" velocity="6.2832"/>
-  </joint>
-  <transmission name="trans_joint_4">
+		<origin rpy="0 0 0" xyz="0.239 0.065 0" />
+		<parent link="link_3" />
+		<child link="link_4" />
+		<axis xyz="1 0 0" />
+		<limit effort="1000" lower="-3.49" upper="3.49" velocity="6.2832" />
+	</joint>
+	<transmission name="trans_joint_4">
 		<type>transmission_interface/SimpleTransmission</type>
 		<joint name="joint_4">
@@ -73,14 +73,14 @@
 			<mechanicalReduction>1</mechanicalReduction>
 		</actuator>
-  </transmission>
+	</transmission>
 	<!--joint_5-->
 	<joint name="joint_5" type="revolute">
-    <origin rpy="0 0 0" xyz="0.141 0 0"/>
-    <parent link="link_4"/>
-    <child link="link_5"/>
-    <axis xyz="0 1 0"/>
-    <limit effort="1000" lower="-2.0071" upper="2.0071" velocity="6.2832"/>
-  </joint>
-  <transmission name="trans_joint_5">
+		<origin rpy="0 0 0" xyz="0.141 0 0" />
+		<parent link="link_4" />
+		<child link="link_5" />
+		<axis xyz="0 1 0" />
+		<limit effort="1000" lower="-2.0071" upper="2.0071" velocity="6.2832" />
+	</joint>
+	<transmission name="trans_joint_5">
 		<type>transmission_interface/SimpleTransmission</type>
 		<joint name="joint_5">
@@ -91,14 +91,14 @@
 			<mechanicalReduction>1</mechanicalReduction>
 		</actuator>
-  </transmission>
+	</transmission>
 	<!--joint_6-->
 	<joint name="joint_6" type="revolute">
-    <origin rpy="0 0 0" xyz="0.065 0 0"/>
-    <parent link="link_5"/>
-    <child link="link_6"/>
-    <axis xyz="1 0 0"/>
-    <limit effort="1000" lower="-6.9813" upper="6.9813" velocity="1"/>
-  </joint>
-  <transmission name="trans_joint_6">
+		<origin rpy="0 0 0" xyz="0.065 0 0" />
+		<parent link="link_5" />
+		<child link="link_6" />
+		<axis xyz="1 0 0" />
+		<limit effort="1000" lower="-6.9813" upper="6.9813" velocity="1" />
+	</joint>
+	<transmission name="trans_joint_6">
 		<type>transmission_interface/SimpleTransmission</type>
 		<joint name="joint_6">
@@ -109,5 +109,5 @@
 			<mechanicalReduction>1</mechanicalReduction>
 		</actuator>
-  </transmission>
+	</transmission>
 	<!-- <xacro:if value="${cam}">
 		<joint name="cam_joint" type="fixed">

Commit message: fixed inertia parameters

File: apc_gripper/urdf/gripper.xacro (robot description, xacro)
@@ -52,5 +52,6 @@
     <inertial>
       <mass value="0.1" />
-      <origin rpy="0 0 0" xyz="-0.031 0 0.04" />
+      <!-- <origin rpy="0 0 0" xyz="-0.031 0 0.04" /> -->
+      <origin rpy="0 0 0" xyz="0 0 0.04" />
       <inertia ixx="0.0000213613" ixy="0" ixz="0" iyy="0.0000595838" iyz="0" izz="0.0000394382" />
     </inertial>
@@ -96,4 +97,5 @@
     <inertial>
       <mass value="0.1" />
+      <origin rpy="0 0 0" xyz="0 0 0.04" />
       <origin rpy="0 0 0" xyz="-0.031 0 0.04" />
       <inertia ixx="0.0000213613" ixy="0" ixz="0" iyy="0.0000595838" iyz="0" izz="0.0000394382" />
