Commit message: effort controllers for grasping

File: apc_gripper/urdf/joints.xacro (robot description, xacro)
@@ -1,65 +1,65 @@
-<?xml version="1.0" ?>
+<?xml version="1.0"?>
 <robot xmlns:xacro="http://ros.org/wiki/xacro">
   <!-- LINKS_BASE JOINTS -->
-    <joint name="gripper_body__left_ext" type="revolute">
-      <axis xyz="1 0 0" />
-      <limit effort="1000" lower="-0.15" upper="0.8" velocity="0.5" />
-      <origin rpy="0 0 0" xyz="0.0 -0.046785 0.103" />
-      <parent link="gripper_body" />
-      <child link="left_ext" />
+  <joint name="gripper_body__left_ext" type="revolute">
+    <axis xyz="1 0 0" />
+    <limit effort="1000" lower="-0.15" upper="0.8" velocity="0.5" />
+    <origin rpy="0 0 0" xyz="0.0 -0.046785 0.103" />
+    <parent link="gripper_body" />
+    <child link="left_ext" />
+  </joint>
+  <transmission name="trans_gripper_body__left_ext">
+    <type>transmission_interface/SimpleTransmission</type>
+    <joint name="gripper_body__left_ext">
+      <hardwareInterface>hardware_interface/EffortJointInterface</hardwareInterface>
     </joint>
-    <transmission name="trans_gripper_body__left_ext">
-  		<type>transmission_interface/SimpleTransmission</type>
-  		<joint name="gripper_body__left_ext">
-  			<hardwareInterface>hardware_interface/PositionJointInterface</hardwareInterface>
-  		</joint>
-  		<actuator name="motor_gripper_body__left_ext">
-  			<hardwareInterface>hardware_interface/PositionJointInterface</hardwareInterface>
-  			<mechanicalReduction>1</mechanicalReduction>
-  		</actuator>
-    </transmission>
-    <joint name="gripper_body__left_int" type="revolute">
-      <axis xyz="1 0 0" />
-      <limit effort="1000" lower="-3.14" upper="3.14" velocity="0.5" />
-      <origin rpy="0 0 0" xyz="0.0 -0.026 0.115" />
-      <parent link="gripper_body" />
-      <child link="left_int" />
-      <mimic joint="gripper_body__left_ext" multiplier="1" offset="0" />
-    </joint>
-    <joint name="gripper_body__right_ext" type="revolute">
-      <axis xyz="1 0 0" />
-      <limit effort="1000" lower="-3.14" upper="3.14" velocity="0.5" />
-      <origin rpy="0 0 3.14" xyz="0 0.046785 0.103" />
-      <parent link="gripper_body" />
-      <child link="right_ext" />
-      <mimic joint="gripper_body__left_ext" multiplier="1" offset="0" />
-    </joint>
-    <joint name="gripper_body__right_int" type="revolute">
-      <axis xyz="1 0 0" />
-      <limit effort="1000" lower="-3.14" upper="3.14" velocity="0.5" />
-      <origin rpy="0 0 0" xyz="0.0 0.026 0.115" />
-      <parent link="gripper_body" />
-      <child link="right_int" />
-      <mimic joint="gripper_body__right_ext" multiplier="-1" offset="0" />
-    </joint>
+    <actuator name="motor_gripper_body__left_ext">
+      <hardwareInterface>hardware_interface/EffortJointInterface</hardwareInterface>
+      <mechanicalReduction>1</mechanicalReduction>
+    </actuator>
+  </transmission>
+  <joint name="gripper_body__left_int" type="revolute">
+    <axis xyz="1 0 0" />
+    <limit effort="1000" lower="-3.14" upper="3.14" velocity="0.5" />
+    <origin rpy="0 0 0" xyz="0.0 -0.026 0.115" />
+    <parent link="gripper_body" />
+    <child link="left_int" />
+    <mimic joint="gripper_body__left_ext" multiplier="1" offset="0" />
+  </joint>
+  <joint name="gripper_body__right_ext" type="revolute">
+    <axis xyz="1 0 0" />
+    <limit effort="1000" lower="-3.14" upper="3.14" velocity="0.5" />
+    <origin rpy="0 0 3.14" xyz="0 0.046785 0.103" />
+    <parent link="gripper_body" />
+    <child link="right_ext" />
+    <mimic joint="gripper_body__left_ext" multiplier="1" offset="0" />
+  </joint>
+  <joint name="gripper_body__right_int" type="revolute">
+    <axis xyz="1 0 0" />
+    <limit effort="1000" lower="-3.14" upper="3.14" velocity="0.5" />
+    <origin rpy="0 0 0" xyz="0.0 0.026 0.115" />
+    <parent link="gripper_body" />
+    <child link="right_int" />
+    <mimic joint="gripper_body__right_ext" multiplier="-1" offset="0" />
+  </joint>
   <!-- FINGERS -->
   <!-- LEFT FINGER -->
-      <joint name="left_ext__left_finger" type="revolute">
-      <axis xyz="1 0 0" />
-      <limit effort="1000" lower="-3.14" upper="3.14" velocity="0.5" />
-      <origin rpy="0 0 0" xyz="0 0 0.080" />
-      <parent link="left_ext" />
-      <child link="left_finger" />
-      <mimic joint="gripper_body__left_ext" multiplier="-1" offset="0" />
-    </joint>
+  <joint name="left_ext__left_finger" type="revolute">
+    <axis xyz="1 0 0" />
+    <limit effort="1000" lower="-3.14" upper="3.14" velocity="0.5" />
+    <origin rpy="0 0 0" xyz="0 0 0.080" />
+    <parent link="left_ext" />
+    <child link="left_finger" />
+    <mimic joint="gripper_body__left_ext" multiplier="-1" offset="0" />
+  </joint>
   <!-- RIGHT FINGER -->
-      <joint name="right_ext__right_finger" type="revolute">
-      <axis xyz="1 0 0" />
-      <limit effort="1000" lower="-3.14" upper="3.14" velocity="0.5" />
-      <origin rpy="0 0 0" xyz="0 0 0.080" />
-      <parent link="right_ext" />
-      <child link="right_finger" />
-      <mimic joint="gripper_body__right_ext" multiplier="-1" offset="0" />
-    </joint>
+  <joint name="right_ext__right_finger" type="revolute">
+    <axis xyz="1 0 0" />
+    <limit effort="1000" lower="-3.14" upper="3.14" velocity="0.5" />
+    <origin rpy="0 0 0" xyz="0 0 0.080" />
+    <parent link="right_ext" />
+    <child link="right_finger" />
+    <mimic joint="gripper_body__right_ext" multiplier="-1" offset="0" />
+  </joint>
   <!-- END - Robot description -->
 </robot>

Commit message: testing position to effort ctrl

File: apc_gripper/urdf/joints.xacro (robot description, xacro)
@@ -5,4 +5,5 @@
     <axis xyz="1 0 0" />
     <limit effort="1000" lower="-0.15" upper="0.8" velocity="0.5" />
+    <!-- <limit effort="3" lower="-0.15" upper="0.8" velocity="0.01" /> -->
     <origin rpy="0 0 0" xyz="0.0 -0.046785 0.103" />
     <parent link="gripper_body" />

Commit message: changed pos control to effort

File: apc_gripper/urdf/joints.xacro (robot description, xacro)
@@ -4,6 +4,6 @@
   <joint name="gripper_body__left_ext" type="revolute">
     <axis xyz="1 0 0" />
-    <limit effort="1000" lower="-0.15" upper="0.8" velocity="0.5" />
-    <!-- <limit effort="3" lower="-0.15" upper="0.8" velocity="0.01" /> -->
+    <!-- <limit effort="1000" lower="-0.15" upper="0.8" velocity="0.5" /> -->
+    <limit effort="1" lower="-0.15" upper="0.8" velocity="0.01" />
     <origin rpy="0 0 0" xyz="0.0 -0.046785 0.103" />
     <parent link="gripper_body" />
@@ -14,7 +14,9 @@
     <joint name="gripper_body__left_ext">
       <hardwareInterface>hardware_interface/EffortJointInterface</hardwareInterface>
+      <!-- <hardwareInterface>hardware_interface/PositionJointInterface</hardwareInterface> -->
     </joint>
     <actuator name="motor_gripper_body__left_ext">
       <hardwareInterface>hardware_interface/EffortJointInterface</hardwareInterface>
+      <!-- <hardwareInterface>hardware_interface/PositionJointInterface</hardwareInterface> -->
       <mechanicalReduction>1</mechanicalReduction>
     </actuator>
