Commit message: update joint limits with real values

File: irb140_sim/urdf/irb140_joints.xacro (robot description, xacro)
@@ -8,5 +8,5 @@
     <child link="link_1"/>
     <axis xyz="0 0 1"/>
-    <limit effort="1000" lower="-0.7853" upper="0.7853" velocity="2.618"/>
+    <limit effort="1000" lower="-3.1416" upper="3.1416" velocity="2.618"/>
   </joint>
   <transmission name="trans_joint_1">
@@ -62,5 +62,5 @@
     <child link="link_4"/>
     <axis xyz="1 0 0"/>
-    <limit effort="1000" lower="-1.4" upper="1.4" velocity="6.2832"/>
+    <limit effort="1000" lower="-3.49" upper="3.49" velocity="6.2832"/>
   </joint>
   <transmission name="trans_joint_4">
@@ -98,5 +98,5 @@
     <child link="link_6"/>
     <axis xyz="1 0 0"/>
-    <limit effort="1000" lower="-1.4" upper="1.4" velocity="1"/>
+    <limit effort="1000" lower="-6.9813" upper="6.9813" velocity="1"/>
   </joint>
   <transmission name="trans_joint_6">

Commit message: added pose command and test gripper

File: irb140_sim/urdf/irb140_joints.xacro (robot description, xacro)
@@ -114,5 +114,5 @@
     <parent link="link_6"/>
     <child link="tool0"/>
-    <origin rpy="0 0 0" xyz="0 0 0"/>
+    <origin rpy="0 1.57 0" xyz="0 0 0"/>
   </joint>
 </robot>

Commit message: edit joint limits for better performance

File: irb140_sim/urdf/irb140_joints.xacro (robot description, xacro)
@@ -26,5 +26,5 @@
     <child link="link_2"/>
     <axis xyz="0 1 0"/>
-    <limit effort="1000" lower="-1.7453" upper="1.7453" velocity="2.618"/>
+    <limit effort="1000" lower="-0.7853" upper="1.5708" velocity="2.618"/>
   </joint>
   <transmission name="trans_joint_2">
@@ -44,5 +44,5 @@
     <child link="link_3"/>
     <axis xyz="0 1 0"/>
-    <limit effort="1000" lower="-2.4434" upper="2.4434" velocity="2.618"/>
+    <limit effort="1000" lower="-2.4434" upper="0.8726" velocity="2.618"/>
   </joint>
   <transmission name="trans_joint_3">

Commit message: minor changes, new gazebo world

File: irb140_sim/urdf/irb140_joints.xacro (robot description, xacro)
@@ -136,5 +136,5 @@
 		<parent link="link_6"/>
 		<child link="tcp_link"/>
-		<origin rpy="0 0 0" xyz="0.21 0 0"/>
+		<origin rpy="0 0 0" xyz="0.24 0 0"/>
 	</joint>
 </robot>
