Commit message: added kinect sim support

File: irb140_sim/urdf/irb140.xacro (robot description, xacro)
@@ -188,6 +188,15 @@
 		</inertial>
 	</link>
+	<!--link_camera-->
+	<link name="cam_link">
+		<visual>
+			<origin rpy="0 0 0" xyz="0 0 0"/>
+			<geometry>
+				<mesh filename="package://irb140_sim/meshes/kinect/meshes/kinect.dae" scale="1 1 1"/>
+			</geometry>
+		</visual>
+	</link>
 	<!--link_tool-->
-	<link name="tool0"/>
+	<!-- <link name="tool0"/> -->
 	<!-- Used for fixing robot to Gazebo 'base_link' -->
   <link name="world"/>

File: irb140_sim/urdf/irb140_joints.xacro (robot description, xacro)
@@ -110,9 +110,21 @@
 		</actuator>
   </transmission>
+	<!--cam_joint-->
+	<joint name="cam_joint" type="fixed">
+    <parent link="link_4"/>
+    <child link="cam_link"/>
+    <origin rpy="0 0 0" xyz="0 0 0.1"/>
+  </joint>
+	<joint name="cam_depth_joint" type="fixed">
+    <origin xyz="0 0 0" rpy="-1.57 0 -1.57 "/>
+    <parent link="cam_link"/>
+    <child link="cam_depth_link"/>
+  </joint>
+  <link name="cam_depth_link"></link>
 	<!--tool_joint-->
-	<joint name="joint_6-tool0" type="fixed">
+	<!-- <joint name="joint_6-tool0" type="fixed">
     <parent link="link_6"/>
     <child link="tool0"/>
     <origin rpy="0 1.57 0" xyz="0 0 0"/>
-  </joint>
+  </joint> -->
 </robot>

Commit message: added gripper designed for this project

File: irb140_sim/urdf/irb140.xacro (robot description, xacro)
@@ -5,4 +5,5 @@
   <!-- Import all Gazebo-customization elements, including Gazebo colors -->
   <xacro:include filename="$(find irb140_sim)/urdf/irb140.gazebo"/>
+	<xacro:include filename="$(find apc_gripper)/urdf/gripper.xacro"/>
  	<!--LINKS-->
 	<!--base_link-->

File: irb140_sim/urdf/irb140_joints.xacro (robot description, xacro)
@@ -116,4 +116,5 @@
     <origin rpy="0 0 0" xyz="0 0 0.1"/>
   </joint>
+	<!-- fix para la nube de puntos -->
 	<joint name="cam_depth_joint" type="fixed">
     <origin xyz="0 0 0" rpy="-1.57 0 -1.57 "/>
@@ -123,8 +124,8 @@
   <link name="cam_depth_link"></link>
 	<!--tool_joint-->
-	<!-- <joint name="joint_6-tool0" type="fixed">
+	<joint name="joint_6-tool0" type="fixed">
     <parent link="link_6"/>
-    <child link="tool0"/>
+    <child link="gripper_body"/>
     <origin rpy="0 1.57 0" xyz="0 0 0"/>
-  </joint> -->
+  </joint>
 </robot>

Commit message: added different scenes for bin pcking and shelf picking

File: irb140_sim/urdf/irb140.xacro (robot description, xacro)
@@ -1,4 +1,6 @@
 <?xml version="1.0" ?>
 <robot name="abb_irb140" xmlns:xacro="http://ros.org/wiki/xacro">
+	<xacro:arg name="cam" default="0" />
+	<xacro:property name="cam" value="$(arg cam)" />
 	<!-- Macros de links y joints generalizados -->
 	<xacro:include filename="$(find irb140_sim)/urdf/irb140_joints.xacro"/>
@@ -191,12 +193,14 @@
 	</link>
 	<!--link_camera-->
-	<link name="cam_link">
-		<visual>
-			<origin rpy="0 0 0" xyz="0 0 0"/>
-			<geometry>
-				<mesh filename="package://irb140_sim/meshes/kinect/meshes/kinect.dae" scale="1 1 1"/>
-			</geometry>
-		</visual>
-	</link>
+	<xacro:if value="${cam}">
+		<link name="cam_link">
+			<visual>
+				<origin rpy="0 0 0" xyz="0 0 0"/>
+				<geometry>
+					<mesh filename="package://irb140_sim/meshes/kinect/meshes/kinect.dae" scale="1 1 1"/>
+				</geometry>
+			</visual>
+		</link>
+	</xacro:if>
 	<!--link_tool-->
 	<!-- <link name="tool0"/> -->

File: irb140_sim/urdf/irb140_joints.xacro (robot description, xacro)
@@ -110,17 +110,19 @@
 		</actuator>
   </transmission>
-	<!--cam_joint-->
-	<joint name="cam_joint" type="fixed">
-    <parent link="link_4"/>
-    <child link="cam_link"/>
-    <origin rpy="0 0 0" xyz="0 0 0.1"/>
-  </joint>
-	<!-- fix para la nube de puntos -->
-	<joint name="cam_depth_joint" type="fixed">
-    <origin xyz="0 0 0" rpy="-1.57 0 -1.57 "/>
-    <parent link="cam_link"/>
-    <child link="cam_depth_link"/>
-  </joint>
-  <link name="cam_depth_link"></link>
+	<xacro:if value="${cam}">
+		<!--cam_joint-->
+		<joint name="cam_joint" type="fixed">
+	    <parent link="link_4"/>
+	    <child link="cam_link"/>
+	    <origin rpy="0 0 0" xyz="0 0 0.1"/>
+	  </joint>
+		<!-- fix para la nube de puntos -->
+		<joint name="cam_depth_joint" type="fixed">
+	    <origin xyz="0 0 0" rpy="-1.57 0 -1.57 "/>
+	    <parent link="cam_link"/>
+	    <child link="cam_depth_link"/>
+	  </joint>
+	  <link name="cam_depth_link"></link>
+	</xacro:if>
 	<!--tool_joint-->
 	<joint name="joint_6-tool0" type="fixed">

Commit message: created motion planning for bin picking tasks

File: irb140_sim/urdf/irb140.xacro (robot description, xacro)
@@ -203,6 +203,4 @@
 		</link>
 	</xacro:if>
-	<!--link_tool-->
-	<!-- <link name="tool0"/> -->
 	<!-- Used for fixing robot to Gazebo 'base_link' -->
   <link name="world"/>

File: irb140_sim/urdf/irb140_joints.xacro (robot description, xacro)
@@ -131,3 +131,10 @@
     <origin rpy="0 1.57 0" xyz="0 0 0"/>
   </joint>
+	<!-- tcp link -->
+	<link name="tcp_link"/>
+	<joint name="tcp_joint" type="fixed">
+		<parent link="link_6"/>
+		<child link="tcp_link"/>
+		<origin rpy="0 0 0" xyz="0.20 0 0"/>
+	</joint>
 </robot>

Commit message: minor edits

File: irb140_sim/urdf/irb140.xacro (robot description, xacro)
@@ -1,6 +1,4 @@
 <?xml version="1.0" ?>
 <robot name="abb_irb140" xmlns:xacro="http://ros.org/wiki/xacro">
-	<xacro:arg name="cam" default="0" />
-	<xacro:property name="cam" value="$(arg cam)" />
 	<!-- Macros de links y joints generalizados -->
 	<xacro:include filename="$(find irb140_sim)/urdf/irb140_joints.xacro"/>
@@ -8,5 +6,4 @@
   <xacro:include filename="$(find irb140_sim)/urdf/irb140.gazebo"/>
 	<!-- gripper files -->
-	<!-- <xacro:include filename="$(find apc_gripper_position)/urdf/gripper.xacro"/> -->
 	<xacro:include filename="$(find apc_gripper)/urdf/gripper.xacro"/>
  	<!--LINKS-->
@@ -193,15 +190,18 @@
 		</inertial>
 	</link>
-	<!--link_camera-->
-	<xacro:if value="${cam}">
-		<link name="cam_link">
-			<visual>
-				<origin rpy="0 0 0" xyz="0 0 0"/>
-				<geometry>
-					<mesh filename="package://irb140_sim/meshes/kinect/meshes/kinect.dae" scale="1 1 1"/>
-				</geometry>
-			</visual>
-		</link>
-	</xacro:if>
+	<!--tool_joint-->
+	<joint name="joint_6-tool0" type="fixed">
+    <parent link="link_6"/>
+    <child link="gripper_body"/>
+    <origin rpy="0 1.57 0"
+						xyz="0 0 0"/>
+  </joint>
+	<!-- tcp link -->
+	<link name="tcp_link"/>
+	<joint name="tcp_joint" type="fixed">
+		<parent link="link_6"/>
+		<child link="tcp_link"/>
+		<origin rpy="0 0 0" xyz="0.24 0 0"/>
+	</joint>
 	<!-- Used for fixing robot to Gazebo 'base_link' -->
   <link name="world"/>

File: irb140_sim/urdf/irb140_joints.xacro (robot description, xacro)
@@ -110,6 +110,5 @@
 		</actuator>
   </transmission>
-	<xacro:if value="${cam}">
-		<!--cam_joint-->
+	<!-- <xacro:if value="${cam}">
 		<joint name="cam_joint" type="fixed">
 	    <parent link="link_4"/>
@@ -117,5 +116,4 @@
 	    <origin rpy="0 0 0" xyz="0 0 0.1"/>
 	  </joint>
-		<!-- fix para la nube de puntos -->
 		<joint name="cam_depth_joint" type="fixed">
 	    <origin xyz="0 0 0" rpy="-1.57 0 -1.57 "/>
@@ -124,17 +122,4 @@
 	  </joint>
 	  <link name="cam_depth_link"></link>
-	</xacro:if>
-	<!--tool_joint-->
-	<joint name="joint_6-tool0" type="fixed">
-    <parent link="link_6"/>
-    <child link="gripper_body"/>
-    <origin rpy="0 1.57 0" xyz="0 0 0"/>
-  </joint>
-	<!-- tcp link -->
-	<link name="tcp_link"/>
-	<joint name="tcp_joint" type="fixed">
-		<parent link="link_6"/>
-		<child link="tcp_link"/>
-		<origin rpy="0 0 0" xyz="0.24 0 0"/>
-	</joint>
+	</xacro:if> -->
 </robot>

Commit message: gripper definitions moved to top

File: irb140_sim/urdf/irb140.xacro (robot description, xacro)
@@ -1,34 +1,53 @@
-<?xml version="1.0" ?>
+<?xml version="1.0"?>
 <robot name="abb_irb140" xmlns:xacro="http://ros.org/wiki/xacro">
 	<!-- Macros de links y joints generalizados -->
-	<xacro:include filename="$(find irb140_sim)/urdf/irb140_joints.xacro"/>
-  <!-- Import all Gazebo-customization elements, including Gazebo colors -->
-  <xacro:include filename="$(find irb140_sim)/urdf/irb140.gazebo"/>
+	<xacro:include filename="$(find irb140_sim)/urdf/irb140_joints.xacro" />
+	<!-- Import all Gazebo-customization elements, including Gazebo colors -->
+	<xacro:include filename="$(find irb140_sim)/urdf/irb140.gazebo" />
 	<!-- gripper files -->
-	<xacro:include filename="$(find apc_gripper)/urdf/gripper.xacro"/>
- 	<!--LINKS-->
+	<xacro:include filename="$(find apc_gripper)/urdf/gripper.xacro" />
+	<!--tool_joint-->
+	<joint name="joint_6-tool0" type="fixed">
+		<parent link="link_6" />
+		<child link="gripper_body" />
+		<origin rpy="0 1.57 0" xyz="0 0 0" />
+	</joint>
+	<!-- tcp link -->
+	<link name="tcp_link" />
+	<joint name="tcp_joint" type="fixed">
+		<parent link="link_6" />
+		<child link="tcp_link" />
+		<origin rpy="0 0 0" xyz="0.24 0 0" />
+	</joint>
+	<!-- Used for fixing robot to Gazebo 'base_link' -->
+	<link name="world" />
+	<joint name="fixed" type="fixed">
+		<parent link="world" />
+		<child link="base_link" />
+	</joint>
+	<!--LINKS-->
 	<!--base_link-->
 	<link name="base_link">
 		<visual>
-			<origin rpy="0 0 0" xyz="0 0 0"/>
-			<geometry>
-				<mesh filename="package://irb140_sim/meshes/irb140/visual/base_link.stl" scale="0.01 0.01 0.01"/>
-			</geometry>
-			<material name="abb_orange">
-				<color rgba="1 0.43 0 1"/>
-			</material>
-		</visual>
-		<collision>
-			<origin rpy="0 0 0" xyz="0 0 0"/>
-			<geometry>
-				<mesh filename="package://irb140_sim/meshes/irb140/collision_low_poly/base_link.stl" scale="0.01 0.01 0.01"/>
-			</geometry>
-			<material name="yellow">
-				<color rgba="0 1 1 1"/>
-			</material>
-		</collision>
-		<inertial>
-			<mass value="26.36"/>
-			<origin xyz="-0.0820 0.0004 0.0599" rpy="0 0 0"/>
+			<origin rpy="0 0 0" xyz="0 0 0" />
+			<geometry>
+				<mesh filename="package://irb140_sim/meshes/irb140/visual/base_link.stl" scale="0.01 0.01 0.01" />
+			</geometry>
+			<material name="abb_orange">
+				<color rgba="1 0.43 0 1" />
+			</material>
+		</visual>
+		<collision>
+			<origin rpy="0 0 0" xyz="0 0 0" />
+			<geometry>
+				<mesh filename="package://irb140_sim/meshes/irb140/collision_low_poly/base_link.stl" scale="0.01 0.01 0.01" />
+			</geometry>
+			<material name="yellow">
+				<color rgba="0 1 1 1" />
+			</material>
+		</collision>
+		<inertial>
+			<mass value="26.36" />
+			<origin xyz="-0.0820 0.0004 0.0599" rpy="0 0 0" />
 			<inertia ixx="0.222" ixy="0" ixz="0.0156" iyy="0.3553" iyz="0.0017" izz="0.5236" />
 		</inertial>
@@ -37,24 +56,24 @@
 	<link name="link_1">
 		<visual>
-			<origin rpy="0 0 0" xyz="0 0 0"/>
-			<geometry>
-				<mesh filename="package://irb140_sim/meshes/irb140/visual/link_1.stl" scale="0.01 0.01 0.01"/>
-			</geometry>
-			<material name="abb_orange">
-				<color rgba="1 0.43 0 1"/>
-			</material>
-		</visual>
-		<collision>
-			<origin rpy="0 0 0" xyz="0 0 0"/>
-			<geometry>
-				<mesh filename="package://irb140_sim/meshes/irb140/collision_low_poly/link_1.stl" scale="0.01 0.01 0.01"/>
-			</geometry>
-			<material name="yellow">
-				<color rgba="0 1 1 1"/>
-			</material>
-		</collision>
-		<inertial>
-			<mass value="34.56"/>
-			<origin xyz="0.0281 0.0438 0.2634" rpy="0 0 0"/>
+			<origin rpy="0 0 0" xyz="0 0 0" />
+			<geometry>
+				<mesh filename="package://irb140_sim/meshes/irb140/visual/link_1.stl" scale="0.01 0.01 0.01" />
+			</geometry>
+			<material name="abb_orange">
+				<color rgba="1 0.43 0 1" />
+			</material>
+		</visual>
+		<collision>
+			<origin rpy="0 0 0" xyz="0 0 0" />
+			<geometry>
+				<mesh filename="package://irb140_sim/meshes/irb140/collision_low_poly/link_1.stl" scale="0.01 0.01 0.01" />
+			</geometry>
+			<material name="yellow">
+				<color rgba="0 1 1 1" />
+			</material>
+		</collision>
+		<inertial>
+			<mass value="34.56" />
+			<origin xyz="0.0281 0.0438 0.2634" rpy="0 0 0" />
 			<inertia ixx="0.5087" ixy="-0.0014" ixz="-0.0524" iyy="0.4612" iyz="-0.0688" izz="0.4567" />
 		</inertial>
@@ -63,24 +82,24 @@
 	<link name="link_2">
 		<visual>
-			<origin rpy="0 0 0" xyz="-0.07 0 -0.352"/>
-			<geometry>
-				<mesh filename="package://irb140_sim/meshes/irb140/visual/link_2.stl" scale="0.01 0.01 0.01"/>
-			</geometry>
-			<material name="abb_orange">
-				<color rgba="1 0.43 0 1"/>
-			</material>
-		</visual>
-		<collision>
-			<origin rpy="0 0 0" xyz="-0.07 0 -0.352"/>
-			<geometry>
-				<mesh filename="package://irb140_sim/meshes/irb140/collision_low_poly/link_2.stl" scale="0.01 0.01 0.01"/>
-			</geometry>
-			<material name="yellow">
-				<color rgba="0 1 1 1"/>
-			</material>
-		</collision>
-		<inertial>
-			<mass value="15.99"/>
-			<origin xyz="-0.0097 -0.0924 0.1983" rpy="0 0 0"/>
+			<origin rpy="0 0 0" xyz="-0.07 0 -0.352" />
+			<geometry>
+				<mesh filename="package://irb140_sim/meshes/irb140/visual/link_2.stl" scale="0.01 0.01 0.01" />
+			</geometry>
+			<material name="abb_orange">
+				<color rgba="1 0.43 0 1" />
+			</material>
+		</visual>
+		<collision>
+			<origin rpy="0 0 0" xyz="-0.07 0 -0.352" />
+			<geometry>
+				<mesh filename="package://irb140_sim/meshes/irb140/collision_low_poly/link_2.stl" scale="0.01 0.01 0.01" />
+			</geometry>
+			<material name="yellow">
+				<color rgba="0 1 1 1" />
+			</material>
+		</collision>
+		<inertial>
+			<mass value="15.99" />
+			<origin xyz="-0.0097 -0.0924 0.1983" rpy="0 0 0" />
 			<inertia ixx="0.3286" ixy="0.0010" ixz="-0.0038" iyy="0.2775" iyz="0.0379" izz="0.0948" />
 		</inertial>
@@ -89,24 +108,24 @@
 	<link name="link_3">
 		<visual>
-			<origin rpy="0 0 0" xyz="-0.07 0.065 -0.712"/>
-			<geometry>
-				<mesh filename="package://irb140_sim/meshes/irb140/visual/link_3.stl" scale="0.01 0.01 0.01"/>
-			</geometry>
-			<material name="abb_orange">
-				<color rgba="1 0.43 0 1"/>
-			</material>
-		</visual>
-		<collision>
-			<origin rpy="0 0 0" xyz="-0.07 0.065 -0.712"/>
-			<geometry>
-				<mesh filename="package://irb140_sim/meshes/irb140/collision_low_poly/link_3.stl" scale="0.01 0.01 0.01"/>
-			</geometry>
-			<material name="yellow">
-				<color rgba="0 1 1 1"/>
-			</material>
-		</collision>
-		<inertial>
-			<mass value="16.9793"/>
-			<origin xyz="0.0196 0.0725 -0.0057" rpy="0 0 0"/>
+			<origin rpy="0 0 0" xyz="-0.07 0.065 -0.712" />
+			<geometry>
+				<mesh filename="package://irb140_sim/meshes/irb140/visual/link_3.stl" scale="0.01 0.01 0.01" />
+			</geometry>
+			<material name="abb_orange">
+				<color rgba="1 0.43 0 1" />
+			</material>
+		</visual>
+		<collision>
+			<origin rpy="0 0 0" xyz="-0.07 0.065 -0.712" />
+			<geometry>
+				<mesh filename="package://irb140_sim/meshes/irb140/collision_low_poly/link_3.stl" scale="0.01 0.01 0.01" />
+			</geometry>
+			<material name="yellow">
+				<color rgba="0 1 1 1" />
+			</material>
+		</collision>
+		<inertial>
+			<mass value="16.9793" />
+			<origin xyz="0.0196 0.0725 -0.0057" rpy="0 0 0" />
 			<inertia ixx="0.0682" ixy="0.0063" ixz="0.004" iyy="0.1990" iyz="0.0007" izz="0.1823" />
 		</inertial>
@@ -115,24 +134,24 @@
 	<link name="link_4">
 		<visual>
-			<origin rpy="0 0 0" xyz="-0.309 0 -0.712"/>
-			<geometry>
-				<mesh filename="package://irb140_sim/meshes/irb140/visual/link_4.stl" scale="0.01 0.01 0.01"/>
-			</geometry>
-			<material name="abb_orange">
-				<color rgba="1 0.43 0 1"/>
-			</material>
-		</visual>
-		<collision>
-			<origin rpy="0 0 0" xyz="-0.309 0 -0.712"/>
-			<geometry>
-				<mesh filename="package://irb140_sim/meshes/irb140/collision_low_poly/link_4.stl" scale="0.01 0.01 0.01"/>
-			</geometry>
-			<material name="yellow">
-				<color rgba="0 1 1 1"/>
-			</material>
-		</collision>
-		<inertial>
-			<mass value="3.7398"/>
-			<origin xyz="0.0726 -0.0012 -0.0014" rpy="0 0 0"/>
+			<origin rpy="0 0 0" xyz="-0.309 0 -0.712" />
+			<geometry>
+				<mesh filename="package://irb140_sim/meshes/irb140/visual/link_4.stl" scale="0.01 0.01 0.01" />
+			</geometry>
+			<material name="abb_orange">
+				<color rgba="1 0.43 0 1" />
+			</material>
+		</visual>
+		<collision>
+			<origin rpy="0 0 0" xyz="-0.309 0 -0.712" />
+			<geometry>
+				<mesh filename="package://irb140_sim/meshes/irb140/collision_low_poly/link_4.stl" scale="0.01 0.01 0.01" />
+			</geometry>
+			<material name="yellow">
+				<color rgba="0 1 1 1" />
+			</material>
+		</collision>
+		<inertial>
+			<mass value="3.7398" />
+			<origin xyz="0.0726 -0.0012 -0.0014" rpy="0 0 0" />
 			<inertia ixx="0.0073" ixy="0.0004" ixz="-0.0001" iyy="0.0153" iyz="0" izz="0.0172" />
 		</inertial>
@@ -141,24 +160,24 @@
 	<link name="link_5">
 		<visual>
-			<origin rpy="0 0 0" xyz="-0.450 0 -0.712"/>
-			<geometry>
-				<mesh filename="package://irb140_sim/meshes/irb140/visual/link_5.stl" scale="0.01 0.01 0.01"/>
-			</geometry>
-			<material name="abb_orange">
-				<color rgba="1 0.43 0 1"/>
-			</material>
-		</visual>
-		<collision>
-			<origin rpy="0 0 0" xyz="-0.450 0 -0.712"/>
-			<geometry>
-				<mesh filename="package://irb140_sim/meshes/irb140/collision_low_poly/link_5.stl" scale="0.01 0.01 0.01"/>
-			</geometry>
-			<material name="yellow">
-				<color rgba="0 1 1 1"/>
-			</material>
-		</collision>
-		<inertial>
-			<mass value="0.3039"/>
-			<origin xyz="-0.0014 0.0006 -0.0002" rpy="0 0 0"/>
+			<origin rpy="0 0 0" xyz="-0.450 0 -0.712" />
+			<geometry>
+				<mesh filename="package://irb140_sim/meshes/irb140/visual/link_5.stl" scale="0.01 0.01 0.01" />
+			</geometry>
+			<material name="abb_orange">
+				<color rgba="1 0.43 0 1" />
+			</material>
+		</visual>
+		<collision>
+			<origin rpy="0 0 0" xyz="-0.450 0 -0.712" />
+			<geometry>
+				<mesh filename="package://irb140_sim/meshes/irb140/collision_low_poly/link_5.stl" scale="0.01 0.01 0.01" />
+			</geometry>
+			<material name="yellow">
+				<color rgba="0 1 1 1" />
+			</material>
+		</collision>
+		<inertial>
+			<mass value="0.3039" />
+			<origin xyz="-0.0014 0.0006 -0.0002" rpy="0 0 0" />
 			<inertia ixx="0.001" ixy="0" ixz="0" iyy="0.002" iyz="0" izz="0.001" />
 		</inertial>
@@ -167,46 +186,26 @@
 	<link name="link_6">
 		<visual>
-			<origin rpy="0 0 0" xyz="-0.515 0 -0.712"/>
-			<geometry>
-				<mesh filename="package://irb140_sim/meshes/irb140/visual/link_6.stl" scale="0.01 0.01 0.01"/>
-			</geometry>
-			<material name="abb_orange">
-				<color rgba="1 0.43 0 1"/>
-			</material>
-		</visual>
-		<collision>
-			<origin rpy="0 0 0" xyz="-0.515 0 -0.712"/>
-			<geometry>
-				<mesh filename="package://irb140_sim/meshes/irb140/collision_low_poly/link_6.stl" scale="0.01 0.01 0.01"/>
-			</geometry>
-			<material name="yellow">
-				<color rgba="0 1 1 1"/>
-			</material>
-		</collision>
-		<inertial>
-			<mass value="0.0549"/>
-			<origin xyz="-0.013 0 0" rpy="0 0 0"/>
+			<origin rpy="0 0 0" xyz="-0.515 0 -0.712" />
+			<geometry>
+				<mesh filename="package://irb140_sim/meshes/irb140/visual/link_6.stl" scale="0.01 0.01 0.01" />
+			</geometry>
+			<material name="abb_orange">
+				<color rgba="1 0.43 0 1" />
+			</material>
+		</visual>
+		<collision>
+			<origin rpy="0 0 0" xyz="-0.515 0 -0.712" />
+			<geometry>
+				<mesh filename="package://irb140_sim/meshes/irb140/collision_low_poly/link_6.stl" scale="0.01 0.01 0.01" />
+			</geometry>
+			<material name="yellow">
+				<color rgba="0 1 1 1" />
+			</material>
+		</collision>
+		<inertial>
+			<mass value="0.0549" />
+			<origin xyz="-0.013 0 0" rpy="0 0 0" />
 			<inertia ixx="0.00001" ixy="0" ixz="0" iyy="0.00001" iyz="0" izz="0.00001" />
 		</inertial>
 	</link>
-	<!--tool_joint-->
-	<joint name="joint_6-tool0" type="fixed">
-    <parent link="link_6"/>
-    <child link="gripper_body"/>
-    <origin rpy="0 1.57 0"
-						xyz="0 0 0"/>
-  </joint>
-	<!-- tcp link -->
-	<link name="tcp_link"/>
-	<joint name="tcp_joint" type="fixed">
-		<parent link="link_6"/>
-		<child link="tcp_link"/>
-		<origin rpy="0 0 0" xyz="0.24 0 0"/>
-	</joint>
-	<!-- Used for fixing robot to Gazebo 'base_link' -->
-  <link name="world"/>
-  <joint name="fixed" type="fixed">
-    <parent link="world"/>
-    <child link="base_link"/>
-  </joint>
 </robot>
