Commit message: renamed package

File: apc_irb140/urdf/irb140_alter.xacro (robot description, xacro)
@@ -1,17 +1,38 @@
 <?xml version="1.0"?>
 <robot name="abb_irb140" xmlns:xacro="http://ros.org/wiki/xacro">
-	<xacro:arg name="robot_namespace" default="/" />
+	<xacro:arg name="tool" default="0" />
+	<xacro:property name="tool" value="$(arg tool)" />
+	<xacro:arg name="tool_name" default="0" />
+	<xacro:property name="tool_name" value="$(arg tool_name)" />
+	<xacro:arg name="tool_file" default="0" />
+	<xacro:property name="tool_file" value="$(arg tool_file)" />
+	<xacro:arg name="tool_x" default="0" />
+	<xacro:property name="tool_x" value="$(arg tool_x)" />
+	<xacro:arg name="tool_y" default="0" />
+	<xacro:property name="tool_y" value="$(arg tool_y)" />
+	<xacro:arg name="tool_z" default="0" />
+	<xacro:property name="tool_z" value="$(arg tool_z)" />
+	<xacro:arg name="tool_roll" default="0" />
+	<xacro:property name="tool_pitch" value="$(arg tool_pitch)" />
+	<xacro:arg name="tool_pitch" default="0" />
+	<xacro:property name="tool_roll" value="$(arg tool_roll)" />
+	<xacro:arg name="tool_yaw" default="0" />
+	<xacro:property name="tool_yaw" value="$(arg tool_yaw)" />
+	<xacro:arg name="tool_tcp" default="0" />
+	<xacro:property name="tool_tcp" value="$(arg tool_tcp)" />
 	<!-- Macros de links y joints generalizados -->
-	<xacro:include filename="$(find irb140_sim)/urdf/irb140_joints.xacro" />
+	<xacro:include filename="$(find apc_irb140)/urdf/irb140_joints.xacro" />
 	<!-- Import all Gazebo-customization elements, including Gazebo colors -->
-	<xacro:include filename="$(find irb140_sim)/urdf/irb140.gazebo" />
-	<!-- gripper files -->
-	<xacro:include filename="$(find apc_gripper)/urdf/gripper.xacro" />
-	<!--tool_joint-->
-	<joint name="joint_6-tool0" type="fixed">
-		<parent link="link_6" />
-		<child link="gripper_body" />
-		<origin rpy="0 1.57 0" xyz="0 0 0" />
-	</joint>
+	<xacro:include filename="$(find apc_irb140)/urdf/irb140.gazebo" />
+	<xacro:if value="${tool}">
+		<!--tool_joint-->
+		<joint name="joint_6-tool0" type="fixed">
+			<parent link="link_6" />
+			<child link="${tool_name}" />
+			<origin rpy="${tool_roll} ${tool_pitch} ${tool_yaw}" xyz="${tool_x} ${tool_y} ${tool_z}" />
+		</joint>
+		<!-- gripper files -->
+		<xacro:include filename="${tool_file}" />
+	</xacro:if>
 	<!-- tcp link -->
 	<link name="tcp_link" />
@@ -19,5 +40,5 @@
 		<parent link="link_6" />
 		<child link="tcp_link" />
-		<origin rpy="0 0 0" xyz="0.24 0 0" />
+		<origin rpy="0 0 0" xyz="${tool_tcp} 0 0" />
 	</joint>
 	<!-- Used for fixing robot to Gazebo 'base_link' -->
@@ -33,14 +54,14 @@
 			<origin rpy="0 0 0" xyz="0 0 0" />
 			<geometry>
-				<mesh filename="package://irb140_sim/meshes/irb140/visual/base_link.stl" scale="0.01 0.01 0.01" />
-			</geometry>
-			<material name="abb_orange">
-				<color rgba="1 0.43 0 1" />
-			</material>
-		</visual>
-		<collision>
-			<origin rpy="0 0 0" xyz="0 0 0" />
-			<geometry>
-				<mesh filename="package://irb140_sim/meshes/irb140/collision_low_poly/base_link.stl" scale="0.01 0.01 0.01" />
+				<mesh filename="package://apc_irb140/meshes/irb140/visual/base_link.stl" scale="0.01 0.01 0.01" />
+			</geometry>
+			<material name="abb_orange">
+				<color rgba="1 0.43 0 1" />
+			</material>
+		</visual>
+		<collision>
+			<origin rpy="0 0 0" xyz="0 0 0" />
+			<geometry>
+				<mesh filename="package://apc_irb140/meshes/irb140/collision_low_poly/base_link.stl" scale="0.01 0.01 0.01" />
 			</geometry>
 			<material name="yellow">
@@ -59,14 +80,14 @@
 			<origin rpy="0 0 0" xyz="0 0 0" />
 			<geometry>
-				<mesh filename="package://irb140_sim/meshes/irb140/visual/link_1.stl" scale="0.01 0.01 0.01" />
-			</geometry>
-			<material name="abb_orange">
-				<color rgba="1 0.43 0 1" />
-			</material>
-		</visual>
-		<collision>
-			<origin rpy="0 0 0" xyz="0 0 0" />
-			<geometry>
-				<mesh filename="package://irb140_sim/meshes/irb140/collision_low_poly/link_1.stl" scale="0.01 0.01 0.01" />
+				<mesh filename="package://apc_irb140/meshes/irb140/visual/link_1.stl" scale="0.01 0.01 0.01" />
+			</geometry>
+			<material name="abb_orange">
+				<color rgba="1 0.43 0 1" />
+			</material>
+		</visual>
+		<collision>
+			<origin rpy="0 0 0" xyz="0 0 0" />
+			<geometry>
+				<mesh filename="package://apc_irb140/meshes/irb140/collision_low_poly/link_1.stl" scale="0.01 0.01 0.01" />
 			</geometry>
 			<material name="yellow">
@@ -85,5 +106,5 @@
 			<origin rpy="0 0 0" xyz="-0.07 0 -0.352" />
 			<geometry>
-				<mesh filename="package://irb140_sim/meshes/irb140/visual/link_2.stl" scale="0.01 0.01 0.01" />
+				<mesh filename="package://apc_irb140/meshes/irb140/visual/link_2.stl" scale="0.01 0.01 0.01" />
 			</geometry>
 			<material name="abb_orange">
@@ -94,5 +115,5 @@
 			<origin rpy="0 0 0" xyz="-0.07 0 -0.352" />
 			<geometry>
-				<mesh filename="package://irb140_sim/meshes/irb140/collision_low_poly/link_2.stl" scale="0.01 0.01 0.01" />
+				<mesh filename="package://apc_irb140/meshes/irb140/collision_low_poly/link_2.stl" scale="0.01 0.01 0.01" />
 			</geometry>
 			<material name="yellow">
@@ -111,5 +132,5 @@
 			<origin rpy="0 0 0" xyz="-0.07 0.065 -0.712" />
 			<geometry>
-				<mesh filename="package://irb140_sim/meshes/irb140/visual/link_3.stl" scale="0.01 0.01 0.01" />
+				<mesh filename="package://apc_irb140/meshes/irb140/visual/link_3.stl" scale="0.01 0.01 0.01" />
 			</geometry>
 			<material name="abb_orange">
@@ -120,5 +141,5 @@
 			<origin rpy="0 0 0" xyz="-0.07 0.065 -0.712" />
 			<geometry>
-				<mesh filename="package://irb140_sim/meshes/irb140/collision_low_poly/link_3.stl" scale="0.01 0.01 0.01" />
+				<mesh filename="package://apc_irb140/meshes/irb140/collision_low_poly/link_3.stl" scale="0.01 0.01 0.01" />
 			</geometry>
 			<material name="yellow">
@@ -137,5 +158,5 @@
 			<origin rpy="0 0 0" xyz="-0.309 0 -0.712" />
 			<geometry>
-				<mesh filename="package://irb140_sim/meshes/irb140/visual/link_4.stl" scale="0.01 0.01 0.01" />
+				<mesh filename="package://apc_irb140/meshes/irb140/visual/link_4.stl" scale="0.01 0.01 0.01" />
 			</geometry>
 			<material name="abb_orange">
@@ -146,5 +167,5 @@
 			<origin rpy="0 0 0" xyz="-0.309 0 -0.712" />
 			<geometry>
-				<mesh filename="package://irb140_sim/meshes/irb140/collision_low_poly/link_4.stl" scale="0.01 0.01 0.01" />
+				<mesh filename="package://apc_irb140/meshes/irb140/collision_low_poly/link_4.stl" scale="0.01 0.01 0.01" />
 			</geometry>
 			<material name="yellow">
@@ -163,5 +184,5 @@
 			<origin rpy="0 0 0" xyz="-0.450 0 -0.712" />
 			<geometry>
-				<mesh filename="package://irb140_sim/meshes/irb140/visual/link_5.stl" scale="0.01 0.01 0.01" />
+				<mesh filename="package://apc_irb140/meshes/irb140/visual/link_5.stl" scale="0.01 0.01 0.01" />
 			</geometry>
 			<material name="abb_orange">
@@ -172,5 +193,5 @@
 			<origin rpy="0 0 0" xyz="-0.450 0 -0.712" />
 			<geometry>
-				<mesh filename="package://irb140_sim/meshes/irb140/collision_low_poly/link_5.stl" scale="0.01 0.01 0.01" />
+				<mesh filename="package://apc_irb140/meshes/irb140/collision_low_poly/link_5.stl" scale="0.01 0.01 0.01" />
 			</geometry>
 			<material name="yellow">
@@ -189,5 +210,5 @@
 			<origin rpy="0 0 0" xyz="-0.515 0 -0.712" />
 			<geometry>
-				<mesh filename="package://irb140_sim/meshes/irb140/visual/link_6.stl" scale="0.01 0.01 0.01" />
+				<mesh filename="package://apc_irb140/meshes/irb140/visual/link_6.stl" scale="0.01 0.01 0.01" />
 			</geometry>
 			<material name="abb_orange">
@@ -198,5 +219,5 @@
 			<origin rpy="0 0 0" xyz="-0.515 0 -0.712" />
 			<geometry>
-				<mesh filename="package://irb140_sim/meshes/irb140/collision_low_poly/link_6.stl" scale="0.01 0.01 0.01" />
+				<mesh filename="package://apc_irb140/meshes/irb140/collision_low_poly/link_6.stl" scale="0.01 0.01 0.01" />
 			</geometry>
 			<material name="yellow">
@@ -210,3 +231,14 @@
 		</inertial>
 	</link>
+	<!--link_camera-->
+	<!-- <xacro:if value="${cam}">
+		<link name="cam_link">
+			<visual>
+				<origin rpy="0 0 0" xyz="0 0 0"/>
+				<geometry>
+					<mesh filename="package://apc_irb140/meshes/kinect/meshes/kinect.dae" scale="1 1 1"/>
+				</geometry>
+			</visual>
+		</link>
+	</xacro:if> -->
 </robot>
